File: Sattelite Board/Sattelite Board.kicad_pcb (KiCad board)
At the start: 2 copper layers, 13 parts, among them U1 MQ-4, U2 MQ-135-Breakout, U3 HIH-4030-Breakout, U4 TMP36, U5 GY-ML8511-Breakout, U6 MPL3115A2-Breakout, U7 Molex_SL-5, U8 Molex_SL-5

Commit message: Finished rev 1 board
Parts:
- removed U8: Molex_SL-5, MRDT-Connectors:MOLEX_SL_5
- U5: footprint MRDT-Devices:ML8511-Breakout -> MRDT-Devices:GY-ML8511-Breakout
- U7: value Molex_SL-5 -> Molex_SL-10; footprint MRDT-Connectors:MOLEX_SL_5 -> MRDT-Connectors:MOLEX_SL_10
- moved R2 191.3 mm to (244.0, 132.7), turned to 90 degrees
- moved R4 189.7 mm to (244.0, 128.4), turned to 270 degrees
- moved R5 189.2 mm to (244.7, 107.3), turned to 270 degrees
- moved R3 173.3 mm to (227.3, 122.1), turned to 270 degrees
- moved R1 173.1 mm to (227.3, 126.3), turned to 90 degrees
- moved U7 148.0 mm to (226.6, 135.6), turned to 180 degrees
- moved U3 67.5 mm to (243.6, 124.2)
- moved U6 53.1 mm to (248.7, 102.4), turned to 90 degrees
- moved U5 50.8 mm to (248.7, 104.4), turned to 180 degrees
- moved U4 38.9 mm to (234.9, 126.5), turned to 270 degrees
- moved U1 17.4 mm to (234.2, 133.6), turned to 0 degrees
- moved U2 0.51 mm to (212.1, 115.8)
Routing:
- net +5V: track 0.00 -> 55.7 mm, vias 0 -> 1
- net +3V3: track 0.00 -> 46.0 mm
- net Pressure_SDA: track 0.00 -> 45.2 mm, vias 0 -> 1
- net Pressure_SCL: track 0.00 -> 44.9 mm, vias 0 -> 1
- net UV_VOUT: track 0.00 -> 42.3 mm, vias 0 -> 1
- net Humidity_VOUT: track 0.00 -> 25.8 mm, vias 0 -> 1
- net Temp_VOUT: track 0.00 -> 21.8 mm, vias 0 -> 1
- net Ammonia_VOUT: track 0.00 -> 13.2 mm
- net Net-(R3-Pad1): track 0.00 -> 11.7 mm, vias 0 -> 1
- net Methane_VOUT: track 0.00 -> 11.6 mm
- net Net-(R4-Pad1): track 0.00 -> 6.70 mm
- net Net-(U6-Pad1): track 0.00 -> 2.54 mm
- net Net-(R5-Pad2): track 0.00 -> 2.45 mm
- added copper zone on B.Cu, net GND
- added copper zone on F.Cu, net GND
Other:
- board outline added: 44.7 x 69.1 mm
- net class Default: clearance 0.2 -> 0.14986
- rule trace_clearance: 0.2 -> 0.14986
- board text added: "Science Sattelite Board Mars Rover 2018 Missouri S&T Andrew Van Horn"

Commit message: Final Touches before Bard Review
Other:
- board text added: "+3V3"
- board text added: "Ammonia"
- board text added: "Humid"
- board text added: "Methane"
- board text added: "Pressure"
- board text added: "Temp"
- board text added: "UV"
Changed lines of the file:
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@@
     (links 28)
     (no_connects 0)
-    (area 0 0 0 0)
+    (area 204.522287 74.008001 273.839715 160.688001)
     (thickness 1.6)
-    (drawings 13)
+    (drawings 20)
     (tracks 78)
     (zones 0)
@@
   )
   (setup
-    (last_trace_width 0.254)
+    (last_trace_width 0.25)
     (user_trace_width 0.254)
     (trace_clearance 0.14986)
@@
     (mod_text_size 1 1)
     (mod_text_width 0.15)
-    (pad_size 1.524 1.524)
-    (pad_drill 0.762)
+    (pad_size 3.45 3.45)
+    (pad_drill 3.45)
     (pad_to_mask_clearance 0.2)
     (aux_axis_origin 0 0)
@@
     (add_net UV_VOUT)
   )
+  (module MRDT-Devices:GY-ML8511-Breakout (layer F.Cu)
+    (at 248.666 104.394 180)
+    (fp_text reference U5 (at 2.284 0.764 180) (layer F.SilkS) hide
+      (effects (font (size 1 1) (thickness 0.15)))
+    )
+    (fp_text value GY-ML8511-Breakout (at 5.588 0.762 180) (layer F.Fab)
+      (effects (font (size 1 1) (thickness 0.15)))
+    )
+    (fp_line (start 9.398 -4.318) (end 9.398 -2.032) (layer F.SilkS) (width 0.15))
+    (fp_line (start 9.398 -2.032) (end 6.604 -2.032) (layer F.SilkS) (width 0.15))
+    (fp_line (start 6.604 -4.318) (end 6.604 -2.032) (layer F.SilkS) (width 0.15))
+    (fp_line (start 9.398 -4.318) (end 6.604 -4.318) (layer F.SilkS) (width 0.15))
+    (fp_circle (center 9.144 -10.922) (end 8.636 -12.954) (layer F.SilkS) (width 0.15))
+    (fp_line (start 0 0) (end 11.43 0) (layer F.SilkS) (width 0.15))
+    (fp_line (start 11.43 0) (end 11.43 -13.208) (layer F.SilkS) (width 0.15))
+    (fp_line (start 11.43 -13.208) (end 0 -13.208) (layer F.SilkS) (width 0.15))
+    (fp_line (start 0 0) (end 0 -13.208) (layer F.SilkS) (width 0.15))
+    (pad 1 thru_hole circle (at 1.524 -11.684 180) (size 1.524 1.524) (drill 0.889) (layers *.Cu *.Mask)
+      (net 6 +3V3))
+    (pad 2 thru_hole circle (at 1.524 -9.144 180) (size 1.524 1.524) (drill 0.889) (layers *.Cu *.Mask)
+      (net 1 GND))
+    (pad 3 thru_hole circle (at 1.524 -6.604 180) (size 1.524 1.524) (drill 0.889) (layers *.Cu *.Mask)
+      (net 11 UV_VOUT))
+    (pad 4 thru_hole circle (at 1.524 -4.064 180) (size 1.524 1.524) (drill 0.889) (layers *.Cu *.Mask)
+      (net 7 "Net-(R5-Pad2)"))
+    (pad 5 thru_hole circle (at 1.524 -1.524 180) (size 1.524 1.524) (drill 0.889) (layers *.Cu *.Mask))
+  )
   (module MRDT-Devices:TMP36-Breakout (layer F.Cu)
     (at 234.95 126.492 270)
@@
     (pad 6 thru_hole circle (at 1.524 -1.524 90) (size 1.6 1.6) (drill 0.9) (layers *.Cu *.Mask)
       (net 1 GND))
-  )
-  (module MRDT-Devices:GY-ML8511-Breakout (layer F.Cu)
-    (at 248.666 104.394 180)
-    (fp_text reference U5 (at 2.284 0.764 180) (layer F.SilkS) hide
-      (effects (font (size 1 1) (thickness 0.15)))
-    )
-    (fp_text value GY-ML8511-Breakout (at 5.588 0.762 180) (layer F.Fab)
-      (effects (font (size 1 1) (thickness 0.15)))
-    )
-    (fp_line (start 9.398 -4.318) (end 9.398 -2.032) (layer F.SilkS) (width 0.15))
-    (fp_line (start 9.398 -2.032) (end 6.604 -2.032) (layer F.SilkS) (width 0.15))
-    (fp_line (start 6.604 -4.318) (end 6.604 -2.032) (layer F.SilkS) (width 0.15))
-    (fp_line (start 9.398 -4.318) (end 6.604 -4.318) (layer F.SilkS) (width 0.15))
-    (fp_circle (center 9.144 -10.922) (end 8.636 -12.954) (layer F.SilkS) (width 0.15))
-    (fp_line (start 0 0) (end 11.43 0) (layer F.SilkS) (width 0.15))
-    (fp_line (start 11.43 0) (end 11.43 -13.208) (layer F.SilkS) (width 0.15))
-    (fp_line (start 11.43 -13.208) (end 0 -13.208) (layer F.SilkS) (width 0.15))
-    (fp_line (start 0 0) (end 0 -13.208) (layer F.SilkS) (width 0.15))
-    (pad 1 thru_hole circle (at 1.524 -11.684 180) (size 1.524 1.524) (drill 0.889) (layers *.Cu *.Mask)
-      (net 6 +3V3))
-    (pad 2 thru_hole circle (at 1.524 -9.144 180) (size 1.524 1.524) (drill 0.889) (layers *.Cu *.Mask)
-      (net 1 GND))
-    (pad 3 thru_hole circle (at 1.524 -6.604 180) (size 1.524 1.524) (drill 0.889) (layers *.Cu *.Mask)
-      (net 11 UV_VOUT))
-    (pad 4 thru_hole circle (at 1.524 -4.064 180) (size 1.524 1.524) (drill 0.889) (layers *.Cu *.Mask)
-      (net 7 "Net-(R5-Pad2)"))
-    (pad 5 thru_hole circle (at 1.524 -1.524 180) (size 1.524 1.524) (drill 0.889) (layers *.Cu *.Mask))
   )
   (module MRDT-Connectors:MOLEX_SL_10 (layer F.Cu)
@@
       (net 13 Pressure_SDA))
   )
+  (gr_text Humid (at 239.014 120.0404) (layer F.SilkS)
+    (effects (font (size 1.5 1.5) (thickness 0.3)))
+  )
+  (gr_text UV (at 250.444 110.8456 90) (layer F.SilkS)
+    (effects (font (size 1.5 1.5) (thickness 0.3)))
+  )
+  (gr_text Temp (at 238.5568 125.476) (layer F.SilkS)
+    (effects (font (size 1.5 1.5) (thickness 0.3)))
+  )
+  (gr_text Pressure (at 240.7412 94.2848) (layer F.SilkS)
+    (effects (font (size 1.5 1.5) (thickness 0.3)))
+  )
+  (gr_text Ammonia (at 219.2528 124.3584) (layer F.SilkS)
+    (effects (font (size 1.5 1.5) (thickness 0.3)))
+  )
+  (gr_text Methane (at 222.4532 109.22) (layer F.SilkS)
+    (effects (font (size 1.5 1.5) (thickness 0.3)))
+  )
+  (gr_text +3V3 (at 250.444 117.1956 90) (layer F.SilkS)
+    (effects (font (size 1.03 1.03) (thickness 0.2575)))
+  )
   (dimension 29.465095 (width 0.3) (layer F.Fab)
     (gr_text "1.1600 in" (at 226.530069 153.116913 359.5060831) (layer F.Fab)
@@
   (segment (start 228.5492 126.4412) (end 228.5492 134.9248) (width 0.254) (layer F.Cu) (net 2))
   (segment (start 227.33 123.2232) (end 227.33 125.2396) (width 0.254) (layer F.Cu) (net 2))
-  (segment (start 222.758 135.636) (end 222.8088 135.636) (width 0.254) (layer B.Cu) (net 3))
-  (segment (start 222.8088 135.636) (end 227.9904 130.4544) (width 0.254) (layer B.Cu) (net 3))
   (segment (start 227.9904 130.4544) (end 242.5192 130.4544) (width 0.254) (layer B.Cu) (net 3))
   (via (at 242.5192 130.4544) (size 0.6) (drill 0.4) (layers F.Cu B.Cu) (net 3))
   (segment (start 242.5192 130.4544) (end 243.4512 129.5224) (width 0.254) (layer F.Cu) (net 3))
+  (segment (start 222.758 135.636) (end 222.8088 135.636) (width 0.254) (layer B.Cu) (net 3))
+  (segment (start 222.8088 135.636) (end 227.9904 130.4544) (width 0.254) (layer B.Cu) (net 3))
   (segment (start 243.4512 129.5224) (end 243.9924 129.5224) (width 0.254) (layer F.Cu) (net 3))
   (segment (start 243.9924 129.5224) (end 243.9924 131.5896) (width 0.254) (layer F.Cu) (net 3))

Commit message: Created Gerbs
Other:
- board text added: "Sensor Lid, Rev1 Mars Rover, 2018 Missouri S&T Andrew Van Horn"
- board text removed: "Science Sattelite Board Mars Rover 2018 Missouri S&T Andrew Van Horn"
Changed lines of the file:
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@@
     (visible_elements 7FFEFF7F)
     (pcbplotparams
-      (layerselection 0x00030_80000001)
+      (layerselection 0x010f0_80000001)
       (usegerberextensions false)
       (excludeedgelayer true)
@@
       (outputformat 1)
       (mirror false)
-      (drillshape 1)
+      (drillshape 0)
       (scaleselection 1)
-      (outputdirectory ""))
+      (outputdirectory Gerbs/))
   )
   (net 0 "")
@@
   (gr_arc (start 212.09 83.82) (end 208.026 83.82) (angle 90) (layer Edge.Cuts) (width 0.15))
   (gr_line (start 212.09 79.756) (end 248.666 79.756) (angle 90) (layer Edge.Cuts) (width 0.15))
-  (gr_text "Science Sattelite Board\nMars Rover 2018\nMissouri S&T\nAndrew Van Horn" (at 233.426 90.297) (layer B.SilkS)
+  (gr_text "Sensor Lid, Rev1\nMars Rover, 2018\nMissouri S&T\nAndrew Van Horn" (at 233.426 90.297) (layer B.SilkS)
     (effects (font (size 1.5 1.5) (thickness 0.3)) (justify mirror))
   )
